File: hardware/warp-front-panel.kicad_sch (KiCad schematic)
At the start: 25 parts, among them J101 Boot, P101 Debug, P102 CON-SENSOR2, Q101 MOSFET_N_CH, U101 XMC1404, U102 BY25Q128ESSIG(R), X101 16MHz

Commit message: prototype version
Parts:
- added C110, C112: 100nF, C0603F, symbol tinkerforge:C
- added C111: 2.2uF, kicad-libraries:C0603F, symbol tinkerforge:C
- added C113: 100uF, kicad-libraries:C1210, symbol tinkerforge:C
- added R105, R106, R107, R108, R109: 82, kicad-libraries:R0603F, symbol tinkerforge:R
- added R110, R112: 1k, kicad-libraries:R0603F, symbol tinkerforge:R
- added R111, R113: 220, kicad-libraries:R0603F, symbol tinkerforge:R
- added SW101: ~, kicad-libraries:LED_TACT_SW_THT, symbol tinkerforge:LED_TACT_SW_THT
- added U104: ESP-PSRAM64?, kicad-libraries:SO-8, symbol tinkerforge:S25FLXXX
- C109: value 10uF -> 2.2uF; footprint C0603F -> kicad-libraries:C0603F
- P101: footprint kicad-libraries:DEBUG_PAD -> kicad-libraries:TSTP_STL
- Q101: value MOSFET_N_CH -> 2N7002P; footprint (none) -> kicad-libraries:SOT23GDS
- U103: footprint (none) -> kicad-libraries:ZIF_14P_0.5mm
Connections:
- net 3V3: now also P102.3, C110.1, C111.1, C112.1, C113.1, R110.1, R112.1, U104.8 (VCC)
- net BOOT: now also U101.23 (P1.3_IHO); no longer U101.36 (P0.7_IO)
- net DIS-AO: now also R109.2
- net DIS-BL: now also U101.25 (P1.1_IHO)
- net DIS-RESET: now also U101.26 (P1.0_IHO), R110.2
- net GND: now also P102.2, C110.2, C111.2, C112.2, C113.2, SW101.4, U104.4 (VSS)
- net M-CLK: now also RP102.3 (P3), U104.6 (SCLK); no longer RP102.6 (R3)
- net M-MISO: now also RP102.1 (P1), U104.2 (SO/IO1); no longer RP102.8 (R1)
- net M-MOSI: now also RP102.2 (P2), R105.1, U104.5 (SI/IO0); no longer RP102.7 (R2)
- net S-CLK: now also RP101.2 (P2); no longer RP101.7 (R2)
- net S-CS: now also RP101.1 (P1); no longer RP101.8 (R1)
- net S-MISO: now also RP101.4 (P4); no longer RP101.5 (R4)
- net S-MOSI: now also RP101.3 (P3); no longer RP101.6 (R3)
- net at U101.15 (P2.12/AIO): now also R108.1
- net at U101.16 (P2.13/AIO): now also R107.1
- net at U101.4 (P2.1_AIO): now also R106.1
- net nWP: now reaches U102.3 (nWP/IO2)
- net nWP: now also R108.2
- net nHOLD: now reaches U102.7 (nHOLD/IO3)
- net nHOLD: now also R107.2
- net at R101.1: now also U101.36 (P0.7_IO); no longer U101.35 (P0.6_IO)
- net at P102.4: now also RP101.8 (R1); no longer RP101.1 (P1)
- net at P102.5: now also RP101.7 (R2); no longer RP101.2 (P2)
- net at P102.6: now also RP101.6 (R3); no longer RP101.3 (P3)
- net at C114.1, P102.7: now also RP101.5 (R4); no longer RP101.4 (P4)
- net at U101.1 (P4.6_IO): now also RP102.6 (R3); no longer RP102.3 (P3)
- net at U101.2 (P4.7_IO): now also RP102.5 (R4); no longer RP102.4 (P4)
- net at U101.47 (P4.4_IO): now also RP102.8 (R1); no longer RP102.1 (P1)
- net at U101.48 (P4.5_IO): now also RP102.7 (R2); no longer RP102.2 (P2)
- net at P101.1: now also U101.24 (P1.2_IHO); no longer U101.31 (P0.2_IO)
- net at U101.32 (P0.3_IO): now also R105.2
- net at U101.40 (P0.9_IO/RTC_XTAL2): now also R109.1
- net at U101.20 (P1.6_IHO): now also R111.1
- net at U101.21 (P1.5_IHO): now also R113.1
- net SW: now reaches U101.22 (P1.4_IHO)
- net SW: now also R112.2, SW101.2
- net M-CS-MEM renamed M-CS-FLASH
- net M-CS-FLASH: now also RP102.4 (P4); no longer RP102.5 (R4)
- new net: R113.2, SW101.L1
- new net: R111.2, SW101.L2
- new net M-CS-RAM: R106.2, U104.1 (nCS)
- no-connect marks 8 -> 25
Other:
- note added: "23AA04M"
- note added: "Copyright Tinkerforge GmbH 2024. This documentation describes Open Hardware and is licensed under the CERN OHL v. 1.1. You may redistribute and modify this documentation under the terms of the CERN OHL v.1.1. (http://ohwr.org/cernohl). This documentation is distributed WITHOUT ANY EXPRESS OR IMPLIED WARRANTY, INCLUDING OF MERCHANTABILITY, SATISFACTORY QUALITY AND FITNESS FOR A PARTICULAR PURPOSE.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"
- note added: "ER-TFT020-3"
- company: (none) -> Tinkerforge GmbH
- title: (none) -> WARP Front Panel
- moved on the sheet: C101, C102, C103, C104, C105, C106, C107, D101, J101, P101, Q101, R101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
