File: hardware/warp-front-panel.kicad_pcb (KiCad board)
At the start: 4 copper layers, 67.4 x 42 mm, 45 parts, among them J101 Boot, P101 Debug, P102 CON-SENSOR2, Q101 2N7002P, U101 XMC1404, U102 BY25Q128ESSIG(R), U104 ESP-PSRAM64?, X101 16MHz

Commit message: drc
Parts:
- SW101: moved to B.Cu
Connections:
- SW101 pad 2: SW -> GND
- SW101 pad 4: GND -> SW
- SW101 pad L1: Net-(R113-Pad2) -> Net-(R111-Pad2)
- SW101 pad L2: Net-(R111-Pad2) -> Net-(R113-Pad2)
Routing:
- net SW: track 38.7 -> 46.1 mm
Other:
- board text added: "WARP Front Panel 1.1"
- board text removed: "WARP Front Panel 1.0"

Commit message: updated design V1.2
Parts:
- removed C110: 100nF, kicad-libraries:C0603F
- removed the G*** at (154.9, 87.7)
- removed R105, R106: 82, kicad-libraries:R0603F
- removed SW101: ~, kicad-libraries:LED_TACT_SW_THT
- removed U104: ESP-PSRAM64?, kicad-libraries:SO-8
- added G***: LOGO, tf:LogoWARP_15x3, F.Cu at (139.0, 55.9)
- added Pw1: CONN_01X04, tf:pin_array_1x4-P2mm_D1mm, F.Cu at (106.2, 59.6)
- added Pw2: CONN_01X04, tf:pin_array_1x4-P2mm_D1mm, F.Cu at (106.2, 82.4)
- added VAL: CE_5mm, tf:CE_5mm, F.Cu at (163.5, 58.9)
- added VAL: WEEE_7mm, tf:WEEE_7mm, F.Cu at (163.6, 65.0)
- moved Fiducial_Mark 67.8 mm to (107.0, 89.0)
- moved Fiducial_Mark 60.8 mm to (163.0, 79.0)
- moved C107 45.8 mm to (147.7, 77.1), turned to -90 degrees
- moved R108 44.5 mm to (156.8, 72.3)
- moved U102 43.2 mm to (150.4, 73.0)
- moved Fiducial_Mark 38.2 mm to (155.0, 52.0)
- moved R107 32.9 mm to (145.3, 75.6), turned to 90 degrees
- moved R101 32.2 mm to (162.7, 86.2)
- moved D101 29.6 mm to (162.7, 84.7), turned to 0 degrees
- moved C105 26.2 mm to (147.8, 90.0), turned to 180 degrees
- moved J101 25.5 mm to (139.5, 87.8)
- moved C103 23.4 mm to (153.6, 88.4)
- moved C104 23.4 mm to (153.6, 83.0)
- moved X101 23.4 mm to (153.6, 85.7)
- moved U101 23.1 mm to (145.7, 84.4)
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Connections:
- R111 pad 2: Net-(R111-Pad2) -> SW-LED2
- R113 pad 2: Net-(R113-Pad2) -> SW-LED1
- U101 pad 32: Net-(U101B-P0.3_IO) -> unconnected-(U101B-P0.3_IO-Pad32)
- U101 pad 4: Net-(U101D-P2.1_AIO) -> unconnected-(U101D-P2.1_AIO-Pad4)
Routing:
- net M-MOSI: track 65.2 -> 15.7 mm, vias 3 -> 0
- net M-CLK: track 57.8 -> 14.5 mm, vias 4 -> 0
- net M-MISO: track 33.7 -> 5.17 mm, vias 2 -> 0
- net Net-(U101C-P1.6_IHO): track 30.3 -> 58.2 mm
- net Net-(U101D-P2.12/AIO): track 4.71 -> 27.6 mm, vias 0 -> 2
- net 3V3: track 36.8 -> 57.6 mm, vias 16 -> 10
- net Net-(U101B-P0.9_IO/RTC_XTAL2): track 10.3 -> 30.9 mm
- net Net-(U101C-P1.5_IHO): track 42.2 -> 60.9 mm
- net M-CS-FLASH: track 25.9 -> 8.12 mm
- net Net-(U101B-P0.3_IO): track 16.7 -> 0.00 mm
- net S-MOSI: track 15.5 -> 31.6 mm
- net DIS-BL: track 52.4 -> 36.4 mm
- net DIS-AO: track 18.1 -> 3.37 mm
- net S-CLK: track 16.9 -> 30.5 mm
- net Net-(U101D-P2.1_AIO): track 12.5 -> 0.00 mm, vias 2 -> 0
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- added copper zone on F.Cu, net 3V3
Other:
- outline, holes or cut-outs redrawn
- board text added: "Status"
- board text added: "WARP Front Panel 1.2"
- board text added: "warp-charger.com"
- board text removed: "1"
- board text removed: "WARP Front Panel 1.1"
- board text removed: "tinkerforge.com"

Commit message: improve routing
Parts:
- removed R113: 220, kicad-libraries:R0603F
- moved G*** 1.98 mm to (139.0, 57.9)
Connections:
- R108 pad 1: Net-(U101D-P2.12/AIO) -> Net-(U101D-P2.1_AIO)
- U101 pad 15: Net-(U101D-P2.12/AIO) -> unconnected-(U101D-P2.12/AIO-Pad15)
- U101 pad 21: Net-(U101C-P1.5_IHO) -> SW-LED1
- U101 pad 4: unconnected-(U101D-P2.1_AIO-Pad4) -> Net-(U101D-P2.1_AIO)
Routing:
- net GND: track 52.9 -> 185.2 mm, vias 32 -> 207
- net Net-(U101C-P1.5_IHO): track 60.9 -> 0.00 mm, vias 2 -> 0
- net SW-LED1: track 3.32 -> 60.0 mm, vias 0 -> 1
- net Net-(U101D-P2.12/AIO): track 27.6 -> 0.00 mm, vias 2 -> 0
- net Net-(U101D-P2.1_AIO): track 0.00 -> 15.8 mm, vias 0 -> 2
- net Net-(U101B-P0.9_IO/RTC_XTAL2): track 30.9 -> 24.9 mm
- net M-CS-FLASH: track 8.12 -> 5.07 mm
Other:
- outline, holes or cut-outs redrawn

Commit message: changed data resistor values to 4,7Ohm
Parts:
- R102, R107, R108, R109, RP102: value 82 -> 4,7
Changed lines of the file:
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@@
 			(drillshape 0)
 			(scaleselection 1)
-			(outputdirectory "pcb")
+			(outputdirectory "../../../Desktop/Gerber-Prototypen/warp-front-panel-1v1/")
 		)
 	)
@@
 		)
 		(property ki_fp_filters "Pin_Header_Straight_1X04 Pin_Header_Angled_1X04 Socket_Strip_Straight_1X04 Socket_Strip_Angled_1X04")
-		(sheetname "Root")
+		(sheetname "Stammblatt")
 		(sheetfile "warp-front-panel.kicad_sch")
 		(attr through_hole)
@@
 		)
 		(property ki_fp_filters "C?")
-		(sheetname "Root")
+		(sheetname "Stammblatt")
 		(sheetfile "warp-front-panel.kicad_sch")
 		(attr smd)
@@
 		)
 		(property ki_fp_filters "Pin_Header_Straight_1X02 Pin_Header_Angled_1X02 Socket_Strip_Straight_1X02 Socket_Strip_Angled_1X02")
-		(sheetname "Root")
+		(sheetname "Stammblatt")
 		(sheetfile "warp-front-panel.kicad_sch")
 		(attr smd)
@@
 		)
 		(property ki_fp_filters "C?")
-		(sheetname "Root")
+		(sheetname "Stammblatt")
 		(sheetfile "warp-front-panel.kicad_sch")
 		(attr smd)
@@
 		)
 		(property ki_fp_filters "Pin_Header_Straight_1X04 Pin_Header_Angled_1X04 Socket_Strip_Straight_1X04 Socket_Strip_Angled_1X04")
-		(sheetname "Root")
+		(sheetname "Stammblatt")
 		(sheetfile "warp-front-panel.kicad_sch")
 		(attr through_hole)
@@
 			)
 		)
-		(sheetname "Root")
+		(sheetname "Stammblatt")
 		(sheetfile "warp-front-panel.kicad_sch")
 		(attr smd)
@@
 		)
 		(property ki_fp_filters "R? SM0603 SM0805 R?-*")
-		(sheetname "Root")
+		(sheetname "Stammblatt")
 		(sheetfile "warp-front-panel.kicad_sch")
 		(attr smd)
@@
 		)
 		(property ki_fp_filters "C?")
-		(sheetname "Root")
+		(sheetname "Stammblatt")
 		(sheetfile "warp-front-panel.kicad_sch")
 		(attr smd)
@@
 			)
 		)
-		(sheetname "Root")
+		(sheetname "Stammblatt")
 		(sheetfile "warp-front-panel.kicad_sch")
 		(attr smd)
@@
 		)
 		(property ki_fp_filters "C?")
-		(sheetname "Root")
+		(sheetname "Stammblatt")
 		(sheetfile "warp-front-panel.kicad_sch")
 		(attr smd)
@@
 		)
 		(property ki_fp_filters "C?")
-		(sheetname "Root")
+		(sheetname "Stammblatt")
 		(sheetfile "warp-front-panel.kicad_sch")
 		(attr smd)
@@
 		)
 		(property ki_fp_filters "C?")
-		(sheetname "Root")
+		(sheetname "Stammblatt")
 		(sheetfile "warp-front-panel.kicad_sch")
 		(attr smd)
@@
 			)
 		)
-		(property "Value" "82"
+		(property "Value" "4,7"
 			(at 0.05 -0.375 0)
 			(layer "F.Fab")
@@
 		)
 		(property ki_fp_filters "R? SM0603 SM0805 R?-*")
-		(sheetname "Root")
+		(sheetname "Stammblatt")
 		(sheetfile "warp-front-panel.kicad_sch")
 		(attr smd)
@@
 			)
 		)
-		(property "Value" "82"
+		(property "Value" "4,7"
 			(at 0.05 -0.375 180)
 			(layer "F.Fab")
@@
 			)
 		)
+		(property "TFX" ""
+			(at 0 0 180)
+			(unlocked yes)
+			(layer "F.Fab")
+			(hide yes)
+			(effects
+				(font
+					(size 1 1)
+					(thickness 0.15)
+				)
+			)
+		)
 		(property ki_fp_filters "R? SM0603 SM0805 R?-*")
-		(sheetname "Root")
+		(sheetname "Stammblatt")
 		(sheetfile "warp-front-panel.kicad_sch")
 		(attr smd)
@@
 		)
 		(property ki_fp_filters "C?")
-		(sheetname "Root")
+		(sheetname "Stammblatt")
 		(sheetfile "warp-front-panel.kicad_sch")
 		(attr smd)
@@
 			)
 		)
-		(property "Value" "82"
+		(property "Value" "4,7"
 			(at 0.05 -0.375 -90)
 			(layer "F.Fab")
@@
 		)
 		(property ki_fp_filters "R? SM0603 SM0805 R?-*")
-		(sheetname "Root")
+		(sheetname "Stammblatt")
 		(sheetfile "warp-front-panel.kicad_sch")
 		(attr smd)
@@
 			)
 		)
-		(sheetname "Root")
+		(sheetname "Stammblatt")
 		(sheetfile "warp-front-panel.kicad_sch")
 		(attr smd)
@@
 		)
 		(property ki_fp_filters "C?")
-		(sheetname "Root")
+		(sheetname "Stammblatt")
 		(sheetfile "warp-front-panel.kicad_sch")
 		(attr smd)
@@
 		)
 		(property ki_fp_filters "R? SM0603 SM0805 R?-*")
-		(sheetname "Root")
+		(sheetname "Stammblatt")
 		(sheetfile "warp-front-panel.kicad_sch")
 		(attr smd)
@@
 			)
 		)
-		(property "Value" "82"
+		(property "Value" "4,7"
 			(at 0.05 -0.375 180)
 			(layer "F.Fab")
@@
 			)
 		)
+		(property "TFX" ""
+			(at 0 0 180)
+			(unlocked yes)
+			(layer "F.Fab")
+			(hide yes)
+			(effects
+				(font
+					(size 1 1)
+					(thickness 0.15)
+				)
+			)
+		)
 		(property ki_fp_filters "R? SM0603 SM0805 R?-*")
-		(sheetname "Root")
+		(sheetname "Stammblatt")
 		(sheetfile "warp-front-panel.kicad_sch")
 		(attr smd)
@@
 		)
 		(property ki_fp_filters "C?")
-		(sheetname "Root")
+		(sheetname "Stammblatt")
 		(sheetfile "warp-front-panel.kicad_sch")
 		(attr smd)
@@
 			)
 		)
-		(sheetname "Root")
+		(sheetname "Stammblatt")
 		(sheetfile "warp-front-panel.kicad_sch")
 		(attr through_hole)
@@
 		)
 		(property ki_fp_filters "R? SM0603 SM0805 R?-*")
-		(sheetname "Root")
+		(sheetname "Stammblatt")
 		(sheetfile "warp-front-panel.kicad_sch")
 		(attr smd)
@@
 		)
 		(property ki_fp_filters "CON-SENSOR2")
-		(sheetname "Root")
+		(sheetname "Stammblatt")
 		(sheetfile "warp-front-panel.kicad_sch")
 		(attr through_hole)
@@
 			)
 		)
-		(property "Value" "82"
+		(property "Value" "4,7"
 			(at -0.025 -0.45 180)
 			(layer "F.Fab")
@@
 			)
 		)
-		(sheetname "Root")
+		(sheetname "Stammblatt")
 		(sheetfile "warp-front-panel.kicad_sch")
 		(attr smd)
@@
 		)
 		(property ki_fp_filters "R? SM0603 SM0805 R?-*")
-		(sheetname "Root")
+		(sheetname "Stammblatt")
 		(sheetfile "warp-front-panel.kicad_sch")
 		(attr smd)
@@
 			)
 		)
-		(sheetname "Root")
+		(sheetname "Stammblatt")
 		(sheetfile "warp-front-panel.kicad_sch")
 		(attr smd)
@@
 		)
 		(property ki_fp_filters "R? SM0603 SM0805 R?-*")
-		(sheetname "Root")
+		(sheetname "Stammblatt")
 		(sheetfile "warp-front-panel.kicad_sch")
 		(attr smd)
@@
 			)
 		)
-		(sheetname "Root")
+		(property "TFX" "TFX-06-204"
+			(at 0 0 -90)
+			(unlocked yes)
+			(layer "F.Fab")
+			(hide yes)
+			(effects
+				(font
+					(size 1 1)
+					(thickness 0.15)
+				)
+			)
+		)
+		(sheetname "Stammblatt")
 		(sheetfile "warp-front-panel.kicad_sch")
 		(attr smd)
@@
 			)
 		)
-		(sheetname "Root")
+		(sheetname "Stammblatt")
 		(sheetfile "warp-front-panel.kicad_sch")
 		(attr smd)
@@
 		)
 		(property ki_fp_filters "R? SM0603 SM0805 R?-*")
-		(sheetname "Root")
+		(sheetname "Stammblatt")
 		(sheetfile "warp-front-panel.kicad_sch")
 		(attr smd)
@@
 		)
 		(property ki_fp_filters "LED-3MM LED-5MM LED-10MM LED-0603 LED-0805 LED-1206 LEDV")
-		(sheetname "Root")
+		(sheetname "Stammblatt")
 		(sheetfile "warp-front-panel.kicad_sch")
 		(attr smd)
@@
 		)
 		(property ki_fp_filters "C?")
-		(sheetname "Root")
+		(sheetname "Stammblatt")
 		(sheetfile "warp-front-panel.kicad_sch")
 		(attr smd)
@@
 		)
 		(property ki_fp_filters "C?")
-		(sheetname "Root")
+		(sheetname "Stammblatt")
 		(sheetfile "warp-front-panel.kicad_sch")
 		(attr smd)
@@
 		)
 		(property ki_fp_filters "C?")
-		(sheetname "Root")
+		(sheetname "Stammblatt")
 		(sheetfile "warp-front-panel.kicad_sch")
 		(attr smd)
@@
 		)
 		(property ki_fp_filters "C?")
-		(sheetname "Root")
+		(sheetname "Stammblatt")
 		(sheetfile "warp-front-panel.kicad_sch")
 		(attr smd)
@@
 	)
 	(gr_line
+		(start 113.375 92)
+		(end 163.875 50)
+		(stroke
+			(width 0.1)
+			(type default)
+		)
+		(layer "F.Fab")
+	)
+	(gr_line
 		(start 161.075 86.654555)
 		(end 161.075 55.254555)
@@
 		(layer "F.Fab")
 	)
+	(gr_circle
+		(center 133.7 71)
+		(end 133.9 71)
+		(stroke
+			(width 0.2)
+			(type default)
+		)
+		(fill none)
+		(layer "F.Fab")
+	)
 	(gr_line
 		(start 158.675 92)
@@
 		(stroke
 			(width 0.1)
+			(type default)
+		)
+		(layer "F.Fab")
+	)
+	(gr_line
+		(start 113.375 50)
+		(end 163.875 92)
+		(stroke
+			(width 0.1)
